File: cad/electrical/BatteryModuleBoard.brd (EAGLE design)
At the start: 96.9 x 24.9 mm, 11 parts

Commit message: Update pcb component sizes and power connections
Parts:
- turned BAT2_IN to 180 degrees
- turned BATT1_CONN_BO to 0 degrees
- turned BATT1_IN to 180 degrees
- turned BATT2_CONN_BO to 0 degrees
Connections:
- net BATT_MID: now also BAT2_IN.P$2, BATT1_CONN_BO.1, BATT1_IN.P$1, BATT2_CONN_BO.2; no longer BAT2_IN.P$1, BATT1_CONN_BO.2, BATT1_IN.P$2, BATT2_CONN_BO.1
- net GND: now also BATT1_CONN_BO.2, BATT1_IN.P$2; no longer BATT1_CONN_BO.1, BATT1_IN.P$1
- net VOUT_PREFUSE: now also BAT2_IN.P$1, BATT2_CONN_BO.1; no longer BAT2_IN.P$2, BATT2_CONN_BO.2
Routing:
- net BATT_MID: track 10.2 -> 0.08 mm
- net GND: track 7.69 -> 5.13 mm
- net VOUT_PREFUSE: track 42.1 -> 43.2 mm
Other:
- board text added: "Amiiform Power Distribution Board V1.01 - 8/23/2024 Iman Adibnazari Bioinspired Robotics and Design Lab UC San Diego"
- board text removed: "Amiiform Power Distribution Board V1.00 - 8/23/2024 Iman Adibnazari Bioinspired Robotics and Design Lab UC San Diego"
